File: light_module.kicad_sch (KiCad schematic)
At the start: 23 parts, among them J1 Conn_01x03_Pin, J2 Conn_01x03_Pin, U1 AL8860MP

Commit message: round
Parts:
- added JP3, JP4: SolderJumper_3_Open, Jumper:SolderJumper-3_P1.3mm_Open_RoundedPad1.0x1.5mm_NumberLabels, symbol Jumper:SolderJumper_3_Open
Connections:
- net at D3.1 (K): now also D2.2 (A); no longer D7.2 (A)
- net at D6.1 (K): now also D5.2 (A); no longer D2.2 (A)
- net at D6.2 (A): now also D7.1 (K); no longer D8.1 (K)
- net LED_KATHODE: now reaches D2.1 (K)
- net LED_KATHODE: now also JP4.2 (C); no longer D5.2 (A)
- net KATHODE_LED renamed V-_LED
- net V-_LED: now also JP3.3 (B), JP4.3 (B); no longer D7.1 (K)
- net V_LED renamed V+_LED
- net V+_LED: now also JP3.1 (A), JP4.1 (A); no longer D1.2 (A)
- new net: D7.2 (A), D8.1 (K)
- new net LED_ANODE: D1.2 (A), JP3.2 (C)
Other:
- note added: "ACHTUNG: Es gibt keinen Standard welche Polarität der SMD2835 Footprint hat. In KiCAD ist das größere Pad die Kathode (Negativ). Bei vielen LEDs ist es andersherum, man kann sie trotzdem auflöten, ist aber schwieriger."
- note added: "JP3 12 & JP4 32 -> Big Pad Kathode JP3 32 & JP4 12 -> Big Pad Anode"
- moved on the sheet: D2, D6, D7
